Commit message: second commit

File: diffdrive_arduino/description/ros2_control/diffbot.ros2_control.xacro (robot description, xacro)
@@ -7,9 +7,10 @@
         <param name="left_wheel_name">left_wheel_joint</param>
         <param name="right_wheel_name">right_wheel_joint</param>
-        <param name="loop_rate">20</param>
+        <param name="loop_rate">40</param>
         <param name="device">/dev/ttyACM0</param>
         <param name="baud_rate">57600</param>
         <param name="timeout_ms">1000</param>
-        <param name="enc_counts_per_rev">400</param>
+        <param name="right_enc_counts_per_rev">4000</param>
+        <param name="left_enc_counts_per_rev">4000</param>
         <param name="pid_p">20</param>
         <param name="pid_d">12</param>

File: diffdrive_arduino/description/urdf/diffbot_description.urdf.xacro (robot description, xacro)
@@ -2,9 +2,5 @@
 <robot xmlns:xacro="http://www.ros.org/wiki/xacro">
   <xacro:macro name="diffbot" params="prefix">
-  <!-- Constants for robot dimensions -->
   <xacro:property name="PI" value="3.1415926535897931"/>
-  <!--<xacro:property name="base_mass" value="30" />  arbitrary value for base mass
-  <xacro:property name="wheel_mass" value="0.6" />  arbitrary value for wheel mass
-  <xacro:property name="caster_wheel_mass" value="0.2" />  arbitrary value for caster wheel mass -->
   <xacro:property name="base_width" value="0.55" />
   <xacro:property name="base_length" value="0.60" />
@@ -13,37 +9,26 @@
   <xacro:property name="wheel_radius" value="0.055" />
   <xacro:property name="caster_wheel_radius" value="0.055" />
-  <xacro:property name="z_offset" value="${wheel_radius/2}" /> <!-- Space btw top of beam and the each joint -->
-  <!-- Base Footprint -->
-  <link name="${prefix}base_footprint" />
+  <xacro:property name="axle_offset" value="0.10" />
+   <link name="${prefix}base_footprint" />
   <joint name="${prefix}base_joint" type="fixed">
     <parent link="${prefix}base_link"/>
     <child link="${prefix}base_footprint"/>
-    <origin xyz="0 0 -0.055" rpy="0 0 0"/> <!-- z değerini küçük tuttum, istersen değiştir -->
+    <origin xyz="0 0 0" rpy="0 0 0"/>
   </joint>
-  <!-- Base Link -->
   <link name="${prefix}base_link">
     <collision>
-      <origin xyz="0 0 ${base_height/2}" rpy="0 0 0"/>
+      <origin xyz="${base_length/2 - axle_offset} 0 ${base_height/2}" rpy="0 0 0"/>
       <geometry>
-        <box size="${base_width} ${base_length} ${base_height}"/>
+        <box size="${base_length} ${base_width} ${base_height}"/>
       </geometry>
     </collision>
     <visual>
-      <origin xyz="0 0 ${base_height/2}" rpy="0 0 0"/>
+      <origin xyz="${base_length/2 - axle_offset} 0 ${base_height/2}" rpy="0 0 0"/>
       <geometry>
-        <box size="${base_width} ${base_length} ${base_height}"/>
+        <box size="${base_length} ${base_width} ${base_height}"/>
       </geometry>
       <material name="orange"/>
     </visual>
-    <!--<inertial>
-      <origin xyz="0 0 0.12" rpy="0 0 0"/>
-      <mass value="${base_mass}"/>
-      <inertia
-        ixx="${base_mass / 12.0 * (base_length*base_length + base_height*base_height)}" ixy="0.0" ixz="0.0"
-        iyy="${base_mass / 12.0 * (base_height*base_height + base_width*base_width)}" iyz="0.0"
-        izz="${base_mass / 12.0 * (base_width*base_width + base_length*base_length)}"/>
-    </inertial>-->
   </link>
-  <!-- Lidar -->
   <xacro:property name="laser_radius" value="0.05"/>
   <xacro:property name="laser_length" value="0.045"/>
@@ -52,5 +37,5 @@
     <parent link="${prefix}base_link"/>
     <child link="${prefix}laser"/>
-    <origin xyz="0 0 ${laser_origin_z}" rpy="0 0 0"/>
+    <origin xyz="${base_length/2 - axle_offset} 0 ${laser_origin_z}" rpy="0 0 0"/>
   </joint>
   <link name="${prefix}laser">
@@ -68,11 +53,27 @@
       </geometry>
     </collision>
-    <!--<inertial>
-      <origin xyz="0 0 0" rpy="0 0 0"/>
-      <mass value="0.1"/>
-      <inertia ixx="0.0002" ixy="0" ixz="0" iyy="0.0002" iyz="0" izz="0.0002"/>
-    </inertial>-->
   </link>
-  <!-- Left Wheel Joint -->
+  <joint name="${prefix}left_wheel_joint" type="continuous">
+    <parent link="${prefix}base_link"/>
+    <child link="${prefix}left_wheel"/>
+    <origin xyz="0 ${base_width/2} 0" rpy="0 0 0"/>
+    <axis xyz="0 1 0"/>
+    <dynamics damping="0.2"/>
+  </joint>
+  <link name="${prefix}left_wheel">
+    <collision>
+      <origin xyz="0 0 0" rpy="${PI/2} 0 0"/>
+      <geometry>
+        <cylinder length="${wheel_len}" radius="${wheel_radius}"/>
+      </geometry>
+    </collision>
+    <visual>
+      <origin xyz="0 0 0" rpy="${PI/2} 0 0"/>
+      <geometry>
+        <cylinder length="${wheel_len}" radius="${wheel_radius}"/>
+      </geometry>
+      <material name="black"/>
+    </visual>
+  </link>
   <joint name="${prefix}right_wheel_joint" type="continuous">
     <parent link="${prefix}base_link"/>
@@ -82,5 +83,4 @@
     <dynamics damping="0.2"/>
   </joint>
-  <!-- Left Wheel Link -->
   <link name="${prefix}right_wheel">
     <collision>
@@ -97,52 +97,10 @@
       <material name="black"/>
     </visual>
-    <!--<inertial>
-      <origin xyz="0 0 0" rpy="${PI/2} 0 0"/>
-      <mass value="${wheel_mass}"/>
-      <inertia
-        ixx="${wheel_mass / 12.0 * (3*wheel_radius + wheel_len*wheel_len)}" ixy="0.0" ixz="0.0"
-        iyy="${wheel_mass / 12.0 * wheel_radius*wheel_radius}" iyz="0.0"
-        izz="${wheel_mass / 12.0 * wheel_radius*wheel_radius}"/>
-    </inertial>-->
   </link>
-  <!-- Right Wheel Joint -->
-  <joint name="${prefix}left_wheel_joint" type="continuous">
-    <parent link="${prefix}base_link"/>
-    <child link="${prefix}left_wheel"/>
-    <origin xyz="0 ${base_width/2} 0" rpy="0 0 0"/>
-    <axis xyz="0 1 0"/>
-    <dynamics damping="0.2"/>
-  </joint>
-  <!-- Right Wheel Link -->
-  <link name="${prefix}left_wheel">
-    <collision>
-      <origin xyz="0 0 0" rpy="${PI/2} 0 0"/>
-      <geometry>
-        <cylinder length="${wheel_len}" radius="${wheel_radius}"/>
-      </geometry>
-    </collision>
-    <visual>
-      <origin xyz="0 0 0" rpy="${PI/2} 0 0"/>
-      <geometry>
-        <cylinder length="${wheel_len}" radius="${wheel_radius}"/>
-      </geometry>
-      <material name="black"/>
-    </visual>
-    <!--<inertial>
-      <origin xyz="0 0 0" rpy="${PI/2} 0 0"/>
-      <mass value="${wheel_mass}"/>
-      <inertia
-        ixx="${wheel_mass / 12.0 * (3*wheel_radius + wheel_len*wheel_len)}" ixy="0.0" ixz="0.0"
-        iyy="${wheel_mass / 12.0 * wheel_radius*wheel_radius}" iyz="0.0"
-        izz="${wheel_mass / 12.0 * wheel_radius*wheel_radius}"/>
-    </inertial>-->
-  </link>
-  <!-- Caster frontal wheel Joint -->
   <joint name="${prefix}caster_frontal_wheel_joint" type="fixed">
     <parent link="${prefix}base_link"/>
     <child link="${prefix}caster_frontal_wheel"/>
-    <origin xyz="${base_width/2 - caster_wheel_radius} 0 0" rpy="0 0 0"/>
+    <origin xyz="${base_length - axle_offset - caster_wheel_radius} 0 ${-wheel_radius + caster_wheel_radius}" rpy="0 0 0"/>
   </joint>
-  <!-- Caster frontal wheel Link -->
   <link name="${prefix}caster_frontal_wheel">
     <collision>
@@ -159,42 +117,4 @@
       <material name="white"/>
     </visual>
-    <!--<inertial>
-      <origin xyz="0 0 0" rpy="0 0 0"/>
-      <mass value="${caster_wheel_mass}"/>
-      <inertia
-        ixx="${caster_wheel_mass * 0.6 * (caster_wheel_radius * caster_wheel_radius)}" ixy="0.0" ixz="0.0"
-        iyy="${caster_wheel_mass * 0.6 * (caster_wheel_radius * caster_wheel_radius)}" iyz="0.0"
-        izz="${caster_wheel_mass * 0.6 * (caster_wheel_radius * caster_wheel_radius)}"/>
-    </inertial>-->
-  </link>
-  <!-- Caster rear wheel Joint -->
-  <joint name="${prefix}caster_rear_wheel_joint" type="fixed">
-    <parent link="${prefix}base_link"/>
-    <child link="${prefix}caster_rear_wheel"/>
-    <origin xyz="${-base_width/2 + caster_wheel_radius} 0 0" rpy="0 0 0"/>
-  </joint>
-  <!-- Caster rear wheel Link -->
-  <link name="${prefix}caster_rear_wheel">
-    <collision>
-      <origin xyz="0 0 0" rpy="0 0 0"/>
-      <geometry>
-        <sphere radius="${caster_wheel_radius}"/>
-      </geometry>
-    </collision>
-    <visual>
-      <origin xyz="0 0 0" rpy="0 0 0"/>
-      <geometry>
-        <sphere radius="${caster_wheel_radius}"/>
-      </geometry>
-      <material name="white"/>
-    </visual>
-    <!--<inertial>
-      <origin xyz="0 0 0" rpy="0 0 0"/>
-      <mass value="${caster_wheel_mass}"/>
-      <inertia
-        ixx="${caster_wheel_mass * 0.6 * (caster_wheel_radius * caster_wheel_radius)}" ixy="0.0" ixz="0.0"
-        iyy="${caster_wheel_mass * 0.6 * (caster_wheel_radius * caster_wheel_radius)}" iyz="0.0"
-        izz="${caster_wheel_mass * 0.6 * (caster_wheel_radius * caster_wheel_radius)}"/>
-    </inertial> -->
   </link>
   </xacro:macro>
